File: electrical/drone_electrical.kicad_sch (KiCad schematic)
At the start: 0 parts

Commit message: init electrical layout
Parts:
- added BT1: Battery_4S_LiPo_XT30, Autonomous_Drone:AMASS_XT30PW_Horizontal_PTH, symbol Autonomous_Drone:Battery_4S_LiPo_XT30
- added CAM1: Camera_OV9281_MIPI_15Pin, Autonomous_Drone:Arducam_Mini_OV9281_24x25mm, symbol Autonomous_Drone:Camera_OV9281_MIPI_15Pin
- added FC1: Flywoo_Goku_GN745_45A_AIO_V3, Autonomous_Drone:Flywoo_Goku_GN745_AIO_V3, symbol Autonomous_Drone:Flywoo_Goku_GN745_45A_AIO_V3
- added M1, M2, M3, M4: Brushless_Motor_2004, Autonomous_Drone:Motor_Mount_2004_12x12mm_M2, symbol Autonomous_Drone:Brushless_Motor_2004
- added S1: MicoAir_MTF-02P, Autonomous_Drone:MicoAir_MTF-02P_21.6x16mm, symbol Autonomous_Drone:MicoAir_MTF-02P
- added U1: Sensor_ToF_VL53L0X, Autonomous_Drone:Sensor_VL53L0X_Breakout_Header, symbol Autonomous_Drone:Sensor_ToF_VL53L0X
- added U2: Radxa_ZERO_3W, Autonomous_Drone:Radxa_ZERO_3W, symbol Autonomous_Drone:Radxa_ZERO_3W
- added VR1: Flywoo_BEC_5V_12V_2A_V2, Autonomous_Drone:Flywoo_BEC_V2.0_17.5x6.5mm, symbol Autonomous_Drone:Flywoo_BEC_5V_12V_2A_V2
Connections:
- new net: FC1.M3C (M3_C), M3.1 (PHASE_A)
- new net: FC1.M3B (M3_B), M3.2 (PHASE_B)
- new net: FC1.M3A (M3_A), M3.3 (PHASE_C)
- new net: BT1.1 (VBAT+), FC1.1 (BAT+), VR1.1 (VIN_2-6S)
- new net: BT1.2 (GND), FC1.2 (BAT-), VR1.2 (GND_IN)
- new net: U2.2 (+5.0V_IN), VR1.4 (VOUT_5V_12V)
- new net: U2.6 (GND), VR1.5 (GND_OUT)
- new net: FC1.M2C (M2_C), M2.1 (PHASE_A)
- new net: FC1.M2B (M2_B), M2.2 (PHASE_B)
- new net: FC1.M2A (M2_A), M2.3 (PHASE_C)
- new net: FC1.M4C (M4_C), M4.1 (PHASE_A)
- new net: FC1.M4B (M4_B), M4.2 (PHASE_B)
- new net: FC1.M4A (M4_A), M4.3 (PHASE_C)
- new net: FC1.M1C (M1_C), M1.1 (PHASE_A)
- new net: FC1.M1B (M1_B), M1.2 (PHASE_B)
- new net: FC1.M1A (M1_A), M1.3 (PHASE_C)
